Commit message: add camera urdf & gz_bridge for the camera data

File: robo_1_description/urdf/mobile.urdf.xacro (robot description, xacro)
@@ -89,3 +89,9 @@
         <origin xyz="${x/3} 0 -0.05" rpy="0 0 0" />
     </joint>
+    <xacro:include filename="camera.xacro"/>
+    <joint name="camera_joint" type="fixed">
+        <parent link="base_link" />
+        <child link="camera_link" />
+        <origin xyz="${x/2} 0 ${z/2}" rpy="0 0 0" />
+    </joint>
 </robot>

Commit message: add LIDAR sensor gazebo plugin, gz topic,gz bridge to ros /scan

File: robo_1_description/urdf/mobile.urdf.xacro (robot description, xacro)
@@ -90,4 +90,5 @@
     </joint>
     <xacro:include filename="camera.xacro"/>
+    <xacro:include filename="lidar.xacro"/>
     <joint name="camera_joint" type="fixed">
         <parent link="base_link" />
@@ -95,3 +96,8 @@
         <origin xyz="${x/2} 0 ${z/2}" rpy="0 0 0" />
     </joint>
+    <joint name="lidar_base_joint" type="fixed">
+        <parent link="base_link" />
+        <child link="lidar_link" />
+        <origin xyz="${x/3} 0 ${z}" rpy="0 0 0" />
+    </joint>
 </robot>
